Commit message: add urdf for rviz

File: topoquad_description/gazebo/materials.xacro (robot description, xacro)
@@ -4,5 +4,11 @@
 https://github.com/ROBOTIS-GIT/open_manipulator/blob/foxy-devel/open_manipulator_x_description/urdf/materials.xacro
 -->
-<robot>
+<robot name="topoquad" xmlns:xacro="http://www.ros.org/wiki/xacro" >
+<material name="silver">
+  <color rgba="0.300 0.300 0.300 1.000"/>
+</material>
+<material name="light_green">
+  <color rgba="0.55 1.00 0.25 1.00"/>
+</material>
   <material name="black">
     <color rgba="0.0 0.0 0.0 1.0"/>

Commit message: update gazebo

File: topoquad_description/gazebo/materials.xacro (robot description, xacro)
@@ -6,5 +6,5 @@
 <robot name="topoquad" xmlns:xacro="http://www.ros.org/wiki/xacro" >
 <material name="silver">
-  <color rgba="0.300 0.300 0.300 1.000"/>
+  <color rgba="0.900 0.900 0.900 1.000"/>
 </material>
 <material name="light_green">

File: topoquad_description/urdf/topoquad.xacro (robot description, xacro)
@@ -4,387 +4,335 @@
 <xacro:include filename="$(find topoquad_description)/gazebo/topoquad.gazebo" />
 <xacro:include filename="$(find topoquad_description)/urdf/topoquad.trans" />
-<link name="world" />
+<!-- <link name="world" />
 <joint name="world_fixed" type="fixed">
   <parent link="world"/>
   <child link="base_link"/>
-</joint>
+</joint> -->
 <link name="base_link">
+  <visual>
+    <origin xyz="0 0 0" rpy="0 0 0"/>
+    <geometry>
+      <mesh filename="package://topoquad_description/meshes/base_link.stl" scale="0.001 0.001 0.001"/>
+    </geometry>
+    <material name="light_green"/>
+  </visual>
+  <collision>
+    <origin xyz="0 0 0" rpy="0 0 0"/>
+    <geometry>
+      <mesh filename="package://topoquad_description/meshes/base_link.stl" scale="0.001 0.001 0.001"/>
+    </geometry>
+  </collision>
+</link>
+<link name="base_inertia">
   <inertial>
     <origin xyz="-0.00042104482109471097 1.886023652127901e-16 -0.01208876855171899" rpy="0 0 0"/>
-    <mass value="0.12658502927364312"/>
+    <mass value="0.160"/> <!-- mass of base_link and battery -->
     <inertia ixx="0.00016" iyy="0.000158" izz="0.000284" ixy="0.0" iyz="0.0" ixz="-0.0"/>
   </inertial>
-  <visual>
-    <origin xyz="0 0 0" rpy="0 0 0"/>
-    <geometry>
-      <mesh filename="package://topoquad_description/meshes/base_link.stl" scale="0.001 0.001 0.001"/>
+</link>
+<link name="Leg_Hip_Yaw-Hip_Pitch_1">
+  <inertial>
+    <origin xyz="0.008275795980022913 0.008280303512164446 -0.014296773725820186" rpy="0 0 0"/>
+    <mass value="0.030"/>
+    <inertia ixx="3e-06" iyy="3e-06" izz="4e-06" ixy="-1e-06" iyz="0.0" ixz="0.0"/>
+  </inertial>
+  <visual>
+    <origin xyz="-0.044548 -0.044548 -0.0146" rpy="0 0 0"/>
+    <geometry>
+      <mesh filename="package://topoquad_description/meshes/Leg_Hip_Yaw-Hip_Pitch_1.stl" scale="0.001 0.001 0.001"/>
+    </geometry>
+    <material name="dark"/>
+  </visual>
+</link>
+<link name="Leg_Hip_Pitch-Knee_Pitch_1">
+  <inertial>
+    <origin xyz="-0.001830990956208714 0.018387603670428118 2.1720514535412624e-06" rpy="0 0 0"/>
+    <mass value="0.030"/>
+    <inertia ixx="3e-06" iyy="3e-06" izz="5e-06" ixy="-1e-06" iyz="0.0" ixz="-0.0"/>
+  </inertial>
+  <visual>
+    <origin xyz="-0.086267 -0.065761 -0.0001" rpy="0 0 0"/>
+    <geometry>
+      <mesh filename="package://topoquad_description/meshes/Leg_Hip_Pitch-Knee_Pitch_1.stl" scale="0.001 0.001 0.001"/>
+    </geometry>
+    <material name="dark"/>
+  </visual>
+  <collision>
+    <origin xyz="0.02121296 0.04171904  -4.0e-06" rpy="1.5707963267948966 0 0.7853981633974483"/>
+    <geometry>
+      <cylinder radius="0.015" length="0.035"/>
+    </geometry>
+  </collision>
+</link>
+<link name="Leg_Foot_1">
+  <inertial>
+    <origin xyz="0.0002588440546713866 0.020505814748426665 1.7389581104099416e-06" rpy="0 0 0"/>
+    <mass value="0.030"/>
+    <inertia ixx="4e-06" iyy="4e-06" izz="7e-06" ixy="-2e-06" iyz="0.0" ixz="0.0"/>
+  </inertial>
+  <visual>
+    <origin xyz="-0.117733 -0.097227 -9.6e-05" rpy="0 0 0"/>
+    <geometry>
+      <mesh filename="package://topoquad_description/meshes/Leg_Foot_1.stl" scale="0.001 0.001 0.001"/>
+    </geometry>
+    <material name="dark"/>
+  </visual>
+  <collision>
+    <origin xyz="0.03323401 0.05374011 0.0001" rpy="0 0 0"/>
+    <geometry>
+        <sphere radius="0.005"/>
+    </geometry>
+  </collision>
+</link>
+<link name="Leg_Hip_Yaw-Hip_Pitch_2">
+  <inertial>
+    <origin xyz="-0.008280303512164446 0.008275795980022913 -0.014296773725820186" rpy="0 0 0"/>
+    <mass value="0.030"/>
+    <inertia ixx="3e-06" iyy="3e-06" izz="4e-06" ixy="1e-06" iyz="0.0" ixz="-0.0"/>
+  </inertial>
+  <visual>
+    <origin xyz="0.044548 -0.044548 -0.0146" rpy="0 0 0"/>
+    <geometry>
+      <mesh filename="package://topoquad_description/meshes/Leg_Hip_Yaw-Hip_Pitch_2.stl" scale="0.001 0.001 0.001"/>
+    </geometry>
+    <material name="dark"/>
+  </visual>
+</link>
+<link name="Leg_Hip_Pitch-Knee_Pitch_2">
+  <inertial>
+    <origin xyz="-0.018387603506052397 -0.0018309911205844492 3.187606818864236e-06" rpy="0 0 0"/>
+    <mass value="0.030"/>
+    <inertia ixx="3e-06" iyy="3e-06" izz="5e-06" ixy="1e-06" iyz="-0.0" ixz="-0.0"/>
+  </inertial>
+  <visual>
+    <origin xyz="0.065761 -0.086267 -0.0001" rpy="0 0 0"/>
+    <geometry>
+      <mesh filename="package://topoquad_description/meshes/Leg_Hip_Pitch-Knee_Pitch_2.stl" scale="0.001 0.001 0.001"/>
+    </geometry>
+    <material name="dark"/>
+  </visual>
+  <collision>
+    <origin xyz="-0.04171904 0.02121296 4.0e-06" rpy="1.5707963267948966 0 -0.7853981633974483"/>
+    <geometry>
+      <cylinder radius="0.015" length="0.035"/>
+    </geometry>
+  </collision>
+</link>
+<link name="Leg_Foot_2">
+  <inertial>
+    <origin xyz="-0.020505814729665825 0.00025884403591058813 2.872762956151594e-06" rpy="0 0 0"/>
+    <mass value="0.030"/>
+    <inertia ixx="4e-06" iyy="4e-06" izz="7e-06" ixy="2e-06" iyz="-0.0" ixz="-0.0"/>
+  </inertial>
+  <visual>
+    <origin xyz="0.097227 -0.117733 -0.0001" rpy="0 0 0"/>
+    <geometry>
+      <mesh filename="package://topoquad_description/meshes/Leg_Foot_2.stl" scale="0.001 0.001 0.001"/>
+    </geometry>
+    <material name="dark"/>
+  </visual>
+  <collision>
+    <origin xyz="-0.05374011 0.03323401 -0.0001" rpy="0 0 0"/>
+    <geometry>
+        <sphere radius="0.005"/>
+    </geometry>
+  </collision>
+</link>
+<link name="Leg_Hip_Yaw-Hip_Pitch_3">
+  <inertial>
+    <origin xyz="-0.008275795980023051 -0.00828030351216475 -0.01429677372582087" rpy="0 0 0"/>
+    <mass value="0.030"/>
+    <inertia ixx="3e-06" iyy="3e-06" izz="4e-06" ixy="-1e-06" iyz="-0.0" ixz="-0.0"/>
+  </inertial>
+  <visual>
+    <origin xyz="0.044548 0.044548 -0.0146" rpy="0 0 0"/>
+    <geometry>
+      <mesh filename="package://topoquad_description/meshes/Leg_Hip_Yaw-Hip_Pitch_3.stl" scale="0.001 0.001 0.001"/>
+    </geometry>
+    <material name="dark"/>
+  </visual>
+</link>
+<link name="Leg_Hip_Pitch-Knee_Pitch_3">
+  <inertial>
+    <origin xyz="0.0018309909562085613 -0.01838760367042834 2.172051453599064e-06" rpy="0 0 0"/>
+    <mass value="0.030"/>
+    <inertia ixx="3e-06" iyy="3e-06" izz="5e-06" ixy="-1e-06" iyz="-0.0" ixz="0.0"/>
+  </inertial>
+  <visual>
+    <origin xyz="0.086267 0.065761 -0.0001" rpy="0 0 0"/>
+    <geometry>
+      <mesh filename="package://topoquad_description/meshes/Leg_Hip_Pitch-Knee_Pitch_3.stl" scale="0.001 0.001 0.001"/>
+    </geometry>
+    <material name="dark"/>
+  </visual>
+  <collision>
+    <origin xyz="-0.02121296 -0.04171904  -4.0e-06" rpy="1.5707963267948966 0 0.7853981633974483"/>
+    <geometry>
+      <cylinder radius="0.015" length="0.035"/>
+    </geometry>
+  </collision>
+</link>
+<link name="Leg_Foot_3">
+  <inertial>
+    <origin xyz="-0.0002588440546715809 -0.02050581474842711 1.7389581112604982e-06" rpy="0 0 0"/>
+    <mass value="0.030"/>
+    <inertia ixx="4e-06" iyy="4e-06" izz="7e-06" ixy="-2e-06" iyz="-0.0" ixz="-0.0"/>
+  </inertial>
+  <visual>
+    <origin xyz="0.117733 0.097227 -9.6e-05" rpy="0 0 0"/>
+    <geometry>
+      <mesh filename="package://topoquad_description/meshes/Leg_Foot_3.stl" scale="0.001 0.001 0.001"/>
+    </geometry>
+    <material name="dark"/>
+  </visual>
+  <collision>
+    <origin xyz="-0.03323401 -0.05374011 0.0001" rpy="0 0 0"/>
+    <geometry>
+        <sphere radius="0.005"/>
+    </geometry>
+  </collision>
+</link>
+<link name="Leg_Hip_Yaw-Hip_Pitch_4">
+  <inertial>
+    <origin xyz="0.008280303512164737 -0.008275795980023044 -0.014296773725821391" rpy="0 0 0"/>
+    <mass value="0.030"/>
+    <inertia ixx="3e-06" iyy="3e-06" izz="4e-06" ixy="1e-06" iyz="-0.0" ixz="0.0"/>
+  </inertial>
+  <visual>
+    <origin xyz="-0.044548 0.044548 -0.0146" rpy="0 0 0"/>
+    <geometry>
+      <mesh filename="package://topoquad_description/meshes/Leg_Hip_Yaw-Hip_Pitch_4.stl" scale="0.001 0.001 0.001"/>
+    </geometry>
+    <material name="dark"/>
+  </visual>
+</link>
+<link name="Leg_Hip_Pitch-Knee_Pitch_4">
+  <inertial>
+    <origin xyz="0.018387603670428465 0.0018309909562084087 2.172051453060744e-06" rpy="0 0 0"/>
+    <mass value="0.030"/>
+    <inertia ixx="3e-06" iyy="3e-06" izz="5e-06" ixy="1e-06" iyz="0.0" ixz="0.0"/>
+  </inertial>
+  <visual>
+    <origin xyz="-0.065761 0.086267 -0.0001" rpy="0 0 0"/>
+    <geometry>
+      <mesh filename="package://topoquad_description/meshes/Leg_Hip_Pitch-Knee_Pitch_4.stl" scale="0.001 0.001 0.001"/>
+    </geometry>
+    <material name="dark"/>
+  </visual>
+  <collision>
+    <origin xyz="0.04171904 -0.02121296 4.0e-06" rpy="1.5707963267948966 0 -0.7853981633974483"/>
+    <geometry>
+      <cylinder radius="0.015" length="0.035"/>
+    </geometry>
+  </collision>
+</link>
+<link name="Leg_Foot_4">
+  <inertial>
+    <origin xyz="0.020505814748427456 -0.000258844054671567 1.7389581107002638e-06" rpy="0 0 0"/>
+    <mass value="0.030"/>
+    <inertia ixx="4e-06" iyy="4e-06" izz="7e-06" ixy="2e-06" iyz="-0.0" ixz="0.0"/>
+  </inertial>
+  <visual>
+    <origin xyz="-0.097227 0.117733 -9.6e-05" rpy="0 0 0"/>
+    <geometry>
+      <mesh filename="package://topoquad_description/meshes/Leg_Foot_4.stl" scale="0.001 0.001 0.001"/>
+    </geometry>
+    <material name="dark"/>
+  </visual>
+  <collision>
+    <origin xyz="0.05374011 -0.03323401 -0.0001" rpy="0 0 0"/>
+    <geometry>
+        <sphere radius="0.005"/>
+    </geometry>
+  </collision>
+</link>
+<link name="Leg_Base_1">
+  <inertial>
+    <origin xyz="-0.00029446900398619885 -0.00029447062550457676 1.0858331483845456e-10" rpy="0 0 0"/>
+    <mass value="0.005"/>
+    <inertia ixx="1e-06" iyy="1e-06" izz="1e-06" ixy="-0.0" iyz="-0.0" ixz="-0.0"/>
+  </inertial>
+  <visual>
+    <origin xyz="-0.032527 -0.032527 -0.0001" rpy="0 0 0"/>
+    <geometry>
+      <mesh filename="package://topoquad_description/meshes/Leg_Base_1.stl" scale="0.001 0.001 0.001"/>
+    </geometry>
+    <material name="dark"/>
+  </visual>
+</link>
+<link name="Leg_Base_2">
+  <inertial>
+    <origin xyz="0.00029447062550457676 -0.00029446900398619885 1.0858331483845456e-10" rpy="0 0 0"/>
+    <mass value="0.005"/>
+    <inertia ixx="1e-06" iyy="1e-06" izz="1e-06" ixy="0.0" iyz="-0.0" ixz="0.0"/>
+  </inertial>
+  <visual>
+    <origin xyz="0.032527 -0.032527 -0.0001" rpy="0 0 0"/>
+    <geometry>
+      <mesh filename="package://topoquad_description/meshes/Leg_Base_2.stl" scale="0.001 0.001 0.001"/>
+    </geometry>
+    <material name="dark"/>
+  </visual>
+</link>
+<link name="Leg_Base_3">
+  <inertial>
+    <origin xyz="0.00029446900398600456 0.00029447062550432 1.0858305406072702e-10" rpy="0 0 0"/>
+    <mass value="0.005"/>
+    <inertia ixx="1e-06" iyy="1e-06" izz="1e-06" ixy="-0.0" iyz="0.0" ixz="0.0"/>
+  </inertial>
+  <visual>
+    <origin xyz="0.032527 0.032527 -0.0001" rpy="0 0 0"/>
+    <geometry>
+      <mesh filename="package://topoquad_description/meshes/Leg_Base_3.stl" scale="0.001 0.001 0.001"/>
+    </geometry>
+    <material name="dark"/>
+  </visual>
+</link>
+<link name="Leg_Base_4">
+  <inertial>
+    <origin xyz="-0.00029447062550429226 0.0002944690039859907 1.0858305682544256e-10" rpy="0 0 0"/>
+    <mass value="0.005"/>
+    <inertia ixx="1e-06" iyy="1e-06" izz="1e-06" ixy="0.0" iyz="0.0" ixz="-0.0"/>
+  </inertial>
+  <visual>
+    <origin xyz="-0.032527 0.032527 -0.0001" rpy="0 0 0"/>
+    <geometry>
+      <mesh filename="package://topoquad_description/meshes/Leg_Base_4.stl" scale="0.001 0.001 0.001"/>
+    </geometry>
+    <material name="dark"/>
+  </visual>
+</link>
+<link name="Layer_Second_with_Spacer_1">
+  <inertial>
+    <origin xyz="5.017947999737173e-15 -0.00015187607502035533 0.06014814419419935" rpy="0 0 0"/>
+    <mass value="0.085"/>
+    <inertia ixx="0.000113" iyy="0.000114" izz="0.000225" ixy="-0.0" iyz="0.0" ixz="0.0"/>
+  </inertial>
+  <visual>
+    <origin xyz="0.0 -0.0 0.0396" rpy="0 0 0"/>
+    <geometry>
+      <mesh filename="package://topoquad_description/meshes/Layer_Second_with_Spacer_1.stl" scale="0.001 0.001 0.001"/>
     </geometry>
     <material name="light_green"/>
   </visual>
-  <collision>
-    <origin xyz="0 0 0" rpy="0 0 0"/>
-    <geometry>
-      <mesh filename="package://topoquad_description/meshes/base_link.stl" scale="0.001 0.001 0.001"/>
-    </geometry>
-  </collision>
-</link>
-<link name="Leg_Hip_Yaw-Hip_Pitch_1">
-  <inertial>
-    <origin xyz="0.008275795980022913 0.008280303512164446 -0.014296773725820186" rpy="0 0 0"/>
-    <mass value="0.01942791659585585"/>
-    <inertia ixx="3e-06" iyy="3e-06" izz="4e-06" ixy="-1e-06" iyz="0.0" ixz="0.0"/>
-  </inertial>
-  <visual>
-    <origin xyz="-0.044548 -0.044548 -0.0146" rpy="0 0 0"/>
-    <geometry>
-      <mesh filename="package://topoquad_description/meshes/Leg_Hip_Yaw-Hip_Pitch_1.stl" scale="0.001 0.001 0.001"/>
-    </geometry>
-    <material name="silver"/>
-  </visual>
-  <collision>
-    <origin xyz="-0.044548 -0.044548 -0.0146" rpy="0 0 0"/>
-    <geometry>
-      <mesh filename="package://topoquad_description/meshes/Leg_Hip_Yaw-Hip_Pitch_1.stl" scale="0.001 0.001 0.001"/>
-    </geometry>
-  </collision>
-</link>
-<link name="Leg_Hip_Pitch-Knee_Pitch_1">
-  <inertial>
-    <origin xyz="-0.001830990956208714 0.018387603670428118 2.1720514535412624e-06" rpy="0 0 0"/>
-    <mass value="0.01942792309846978"/>
-    <inertia ixx="3e-06" iyy="3e-06" izz="5e-06" ixy="-1e-06" iyz="0.0" ixz="-0.0"/>
-  </inertial>
-  <visual>
-    <origin xyz="-0.086267 -0.065761 -0.0001" rpy="0 0 0"/>
-    <geometry>
-      <mesh filename="package://topoquad_description/meshes/Leg_Hip_Pitch-Knee_Pitch_1.stl" scale="0.001 0.001 0.001"/>
-    </geometry>
-    <material name="silver"/>
-  </visual>
-  <collision>
-    <origin xyz="-0.086267 -0.065761 -0.0001" rpy="0 0 0"/>
-    <geometry>
-      <mesh filename="package://topoquad_description/meshes/Leg_Hip_Pitch-Knee_Pitch_1.stl" scale="0.001 0.001 0.001"/>
-    </geometry>
-  </collision>
-</link>
-<link name="Leg_Foot_1">
-  <inertial>
-    <origin xyz="0.0002588440546713866 0.020505814748426665 1.7389581104099416e-06" rpy="0 0 0"/>
-    <mass value="0.021556207825352915"/>
-    <inertia ixx="4e-06" iyy="4e-06" izz="7e-06" ixy="-2e-06" iyz="0.0" ixz="0.0"/>
-  </inertial>
-  <visual>
-    <origin xyz="-0.117733 -0.097227 -9.6e-05" rpy="0 0 0"/>
-    <geometry>
-      <mesh filename="package://topoquad_description/meshes/Leg_Foot_1.stl" scale="0.001 0.001 0.001"/>
-    </geometry>
-    <material name="silver"/>
-  </visual>
-  <collision>
-    <origin xyz="-0.117733 -0.097227 -9.6e-05" rpy="0 0 0"/>
-    <geometry>
-      <mesh filename="package://topoquad_description/meshes/Leg_Foot_1.stl" scale="0.001 0.001 0.001"/>
-    </geometry>
-  </collision>
-</link>
-<link name="Leg_Hip_Yaw-Hip_Pitch_2">
-  <inertial>
-    <origin xyz="-0.008280303512164446 0.008275795980022913 -0.014296773725820186" rpy="0 0 0"/>
-    <mass value="0.01942791659585585"/>
-    <inertia ixx="3e-06" iyy="3e-06" izz="4e-06" ixy="1e-06" iyz="0.0" ixz="-0.0"/>
-  </inertial>
-  <visual>
-    <origin xyz="0.044548 -0.044548 -0.0146" rpy="0 0 0"/>
-    <geometry>
-      <mesh filename="package://topoquad_description/meshes/Leg_Hip_Yaw-Hip_Pitch_2.stl" scale="0.001 0.001 0.001"/>
-    </geometry>
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